File: KiCad/Temperature-controller-with-ESP8266/Temperature-controller-with-ESP8266.sch (KiCad schematic (older format))
At the start: 48 parts, among them J1 RJ13, J3 USB_B_Micro, J4 Conn_01x08_Female, J5 Conn_01x08_Female, J8 Screw_Terminal_01x02, J9 Screw_Terminal_01x03, Q1 S8050, Q2 S8050, Q4 MMBT5551L, SW1 SW_Push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

Commit message: zaloha
Connections:
- net GND: no longer SW2.2 (B)
Changed lines of the file:
@@
 	1    0    0    -1
 $EndComp
-$Comp
-L power:GND #PWR022
-U 1 1 5FB16CF7
-P 3400 4750
-F 0 "#PWR022" H 3400 4500 50  0001 C CNN
-F 1 "GND" H 3405 4577 50  0000 C CNN
-F 2 "" H 3400 4750 50  0001 C CNN
-F 3 "" H 3400 4750 50  0001 C CNN
-	1    3400 4750
-	1    0    0    -1
-$EndComp
-Wire Wire Line
-	3400 4750 3400 4600
 Text GLabel 3200 4100 0    50   Input ~ 0
 BUTTON
@@
 Wire Notes Line
 	500  5200 5800 5200
-Text Notes 600  5400 0    50   ~ 0
+Text Notes 650  5400 0    50   ~ 0
 USB TO UART
 Wire Notes Line
