File: KiCad/Temperature-controller-with-ESP8266_v2_all/Temperature-controller-with-ESP8266.sch (KiCad schematic (older format))
At the start: 59 parts, among them J1 USB_B_Micro, J10 Conn_01x08_Male, J2 Conn_01x04_Male, J3 Conn_01x04_Female, J4 Conn_01x03_Male, J5 RJ13, J6 Conn_01x03_Male, J7 Screw_Terminal_01x02, J8 Screw_Terminal_01x02, J9 Conn_01x08_Male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

Commit message: Test of Git+ module atom
Connections:
- net GPIO016 is gone; now on net BUTTON: U1.4 (GPIO16)
Changed lines of the file:
@@
 BUTTON
 Text GLabel 3350 3000 2    50   Input ~ 0
-GPIO016
+GPIO16
 Wire Wire Line
 	3350 3000 3150 3000
