File: KiCad/Temperature-controller-with-ESP8266_v2_part2/Temperature-controller-with-ESP8266.kicad_pcb (KiCad board)
At the start: 2 copper layers, 45.6 x 63.5 mm, 41 parts, among them J1 USB_B_Micro, J10 Conn_01x08_Male, J2 Conn_01x04_Male, J4 Conn_01x03_Male, J5 RJ13, J6 Conn_01x03_Male, J9 Conn_01x08_Male, Q1 SS8050-H, Q2 SS8050-H, SW1 SW_Push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

Commit message: Test of Git+ module atom
Parts:
- added D5: LED, LED_THT:LED_D3.0mm, F.Cu at (139.7, 74.8)
- added G***: LOGO, Symbol:vut_fekt_small, F.Cu at (154.7, 112.1)
- added G***: LOGO, Symbol:logo, B.Cu at (136.1, 99.8)
- added Q5: SS8050-H, Package_TO_SOT_SMD:SOT-23, F.Cu at (134.9, 70.0)
- added R18: 500, Resistor_SMD:R_0805_2012Metric, F.Cu at (135.0, 76.1)
- added R19: 200, Resistor_SMD:R_0805_2012Metric, F.Cu at (142.0, 76.2)
- R11: value R -> 1k
- moved R9 27.0 mm to (117.5, 97.8)
- moved R15 8.13 mm to (148.6, 74.8)
- moved R17 6.91 mm to (145.8, 86.6), turned to 90 degrees
- moved R16 6.76 mm to (148.2, 85.7), turned to 90 degrees
- moved R14 5.36 mm to (148.5, 70.2)
- moved R11 5.03 mm to (129.8, 69.8), turned to 270 degrees
- moved SW2 4.29 mm to (121.4, 65.9)
- moved C3 4.15 mm to (128.3, 80.8), turned to 270 degrees
- moved J5 3.92 mm to (142.7, 68.1)
- moved J4 3.29 mm to (154.8, 71.6)
- moved J6 3.29 mm to (152.3, 71.6)
- moved C4 2.90 mm to (115.8, 71.6)
- moved U5 2.87 mm to (124.1, 73.4)
- moved D1 2.29 mm to (133.0, 74.7), turned to 180 degrees
- moved R1 2.24 mm to (117.5, 88.4)
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Connections:
- J4 pad 1: ADC -> +3V3
- J4 pad 2: +3V3 -> ADC
- J6 pad 1: DATA -> +3V3
- J6 pad 2: +3V3 -> DATA
- R11 pad 1: +5V -> Net-(Q5-Pad1)
- R11 pad 2: Net-(D1-Pad2) -> GPIO13
- SW2 pad 3: Net-(D1-Pad1) -> (no net)
- U1 pad 4: (no net) -> BUTTON
Routing:
- net GPIO15: track 28.2 -> 112.3 mm, vias 0 -> 2
- net GPIO13: track 4.43 -> 40.4 mm, vias 0 -> 1
- net GND: track 27.3 -> 57.4 mm, vias 17 -> 15
- net Net-(D1-Pad1): track 24.9 -> 4.49 mm, vias 1 -> 0
- net GPIO4: track 45.1 -> 25.9 mm, vias 1 -> 0
- net DATA: track 57.0 -> 68.3 mm
- net +5V: track 110.4 -> 117.6 mm, vias 0 -> 1
- net Net-(Q5-Pad1): track 0.00 -> 6.98 mm
- net DTR: track 32.2 -> 27.1 mm
- net BUTTON: track 48.6 -> 43.6 mm
- net GPIO5: track 27.2 -> 22.3 mm, vias 1 -> 0
- net Net-(D1-Pad2): track 4.53 -> 7.56 mm
- net ADC: track 43.0 -> 45.9 mm, vias 1 -> 2
- net RTS: track 31.3 -> 28.7 mm
- net Net-(D5-Pad1): track 0.00 -> 2.49 mm
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Other:
- board size 45.6 x 63.5 mm -> 45.6 x 59.6 mm
- board text added: "ESP-12F"
- board text added: "HC340G"
- board text added: "M24512"
- board text added: "xvymaz11@vutbr.cz"
