File: KiCad/Temperature-controller-with-ESP8266_v2_part2/Temperature-controller-with-ESP8266.sch (KiCad schematic (older format))
At the start: 59 parts, among them J1 USB_B_Micro, J10 Conn_01x08_Male, J2 Conn_01x04_Male, J3 Conn_01x04_Female, J4 Conn_01x03_Male, J5 RJ13, J6 Conn_01x03_Male, J7 Screw_Terminal_01x02, J8 Screw_Terminal_01x02, J9 Conn_01x08_Male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

Commit message: Test of Git+ module atom
Parts:
- added D5: LED, LED_THT:LED_D3.0mm, symbol Device:LED
- added Q5: SS8050-H, Package_TO_SOT_SMD:SOT-23, symbol Device:Q_NPN_BEC
- added R18: 500, Resistor_SMD:R_0805_2012Metric, symbol Device:R
- added R19: 200, Resistor_SMD:R_0805_2012Metric, symbol Device:R
- R11: value R -> 1k
Connections:
- net GPIO016 is gone; now on net BUTTON: U1.4 (GPIO16)
- net +3V3: now also J4.1 (Pin_1), J6.1 (Pin_1); no longer J4.2 (Pin_2), J6.2 (Pin_2)
- net +5V: now also R18.1; no longer R11.1
- net ADC: now also J4.2 (Pin_2); no longer J4.1 (Pin_1)
- net DATA: now also J6.2 (Pin_2); no longer J6.1 (Pin_1)
- net GND: now also Q5.2 (E), R19.2
- net GPIO13: now also R11.2
- net GPIO15: now also D5.2 (A)
- net at SW2.3 (C): no longer D1.1 (K)
- net at D1.2 (A): now also R18.2; no longer R11.2
- new net: Q5.1 (B), R11.1
- new net: D1.1 (K), Q5.3 (C)
- new net: D5.1 (K), R19.1
Other:
- moved on the sheet: R1, R10, R2, R7, R8, R9, SW1, SW2, U1

Commit message: Zaloha 23.05.2021
Parts:
- D1: value LED -> LED Green
- D2: value LED -> LED red
- D5: value LED -> LED Yellow
- R1, R10, R2, R7: value 10k -> 20k
- R15: value 150 -> 470
- R18: value 500 -> 1k2
- R19: value 200 -> 2k
- R8: value R -> 20k
Other:
- moved on the sheet: D5, R19, R9
Changed lines of the file:
@@
 P 1250 1950
 F 0 "R2" V 1100 1950 50  0000 C CNN
-F 1 "10k" V 1000 1950 50  0000 C CNN
+F 1 "20k" V 1000 1950 50  0000 C CNN
 F 2 "Resistor_SMD:R_0805_2012Metric" V 1180 1950 50  0001 C CNN
 F 3 "~" H 1250 1950 50  0001 C CNN
@@
 P 1250 1750
 F 0 "R1" V 1043 1750 50  0000 C CNN
-F 1 "10k" V 1134 1750 50  0000 C CNN
+F 1 "20k" V 1134 1750 50  0000 C CNN
 F 2 "Resistor_SMD:R_0805_2012Metric" V 1180 1750 50  0001 C CNN
 F 3 "~" H 1250 1750 50  0001 C CNN
@@
 P 5250 1300
 F 0 "R7" V 5043 1300 50  0000 C CNN
-F 1 "10k" V 5134 1300 50  0000 C CNN
+F 1 "20k" V 5134 1300 50  0000 C CNN
 F 2 "Resistor_SMD:R_0805_2012Metric" V 5180 1300 50  0001 C CNN
 F 3 "~" H 5250 1300 50  0001 C CNN
@@
 P 4750 1300
 F 0 "R10" V 4543 1300 50  0000 C CNN
-F 1 "10k" V 4634 1300 50  0000 C CNN
+F 1 "20k" V 4634 1300 50  0000 C CNN
 F 2 "Resistor_SMD:R_0805_2012Metric" V 4680 1300 50  0001 C CNN
 F 3 "~" H 4750 1300 50  0001 C CNN
@@
 L Device:R R9
 U 1 1 5FA2E6E4
-P 3900 1300
-F 0 "R9" V 3693 1300 50  0000 C CNN
-F 1 "10k" V 3784 1300 50  0000 C CNN
-F 2 "Resistor_SMD:R_0805_2012Metric" V 3830 1300 50  0001 C CNN
-F 3 "~" H 3900 1300 50  0001 C CNN
-	1    3900 1300
+P 3700 1300
+F 0 "R9" V 3493 1300 50  0000 C CNN
+F 1 "10k" V 3584 1300 50  0000 C CNN
+F 2 "Resistor_SMD:R_0805_2012Metric" V 3630 1300 50  0001 C CNN
+F 3 "~" H 3700 1300 50  0001 C CNN
+	1    3700 1300
 	1    0    0    -1
 $EndComp
@@
 L power:GND #PWR017
 U 1 1 5FA36946
-P 3900 1600
-F 0 "#PWR017" H 3900 1350 50  0001 C CNN
-F 1 "GND" H 3905 1427 50  0000 C CNN
-F 2 "" H 3900 1600 50  0001 C CNN
-F 3 "" H 3900 1600 50  0001 C CNN
-	1    3900 1600
+P 3700 1600
+F 0 "#PWR017" H 3700 1350 50  0001 C CNN
+F 1 "GND" H 3705 1427 50  0000 C CNN
+F 2 "" H 3700 1600 50  0001 C CNN
+F 3 "" H 3700 1600 50  0001 C CNN
+	1    3700 1600
 	1    0    0    -1
 $EndComp
 Text GLabel 5250 1000 1    50   Input ~ 0
 GPIO0
-Text GLabel 3900 1000 1    50   Input ~ 0
+Text GLabel 3700 1000 1    50   Input ~ 0
 GPIO15
 Text GLabel 950  2150 0    50   Input ~ 0
@@
 P 5100 2600
 F 0 "R8" H 5170 2646 50  0000 L CNN
-F 1 "R" H 5170 2555 50  0000 L CNN
+F 1 "20k" H 5170 2555 50  0000 L CNN
 F 2 "Resistor_SMD:R_0805_2012Metric" V 5030 2600 50  0001 C CNN
 F 3 "~" H 5100 2600 50  0001 C CNN
@@
 P 7500 2650
 F 0 "R15" H 7570 2696 50  0000 L CNN
-F 1 "150" H 7570 2605 50  0000 L CNN
+F 1 "470" H 7570 2605 50  0000 L CNN
 F 2 "Resistor_SMD:R_0805_2012Metric" V 7430 2650 50  0001 C CNN
 F 3 "~" H 7500 2650 50  0001 C CNN
@@
 P 7500 2950
 F 0 "D2" V 7539 2832 50  0000 R CNN
-F 1 "LED" V 7448 2832 50  0001 R CNN
+F 1 "LED red" V 7448 2832 50  0000 R CNN
 F 2 "LED_THT:LED_D3.0mm" H 7500 2950 50  0001 C CNN
 F 3 "~" H 7500 2950 50  0001 C CNN
@@
 P 3900 2900
 F 0 "D1" V 3939 2782 50  0000 R CNN
-F 1 "LED" V 3848 2782 50  0000 R CNN
+F 1 "LED Green" V 3848 2782 50  0000 R CNN
 F 2 "LED_THT:LED_D3.0mm" H 3900 2900 50  0001 C CNN
 F 3 "~" H 3900 2900 50  0001 C CNN
@@
 P 3900 2600
 F 0 "R18" V 3693 2600 50  0000 C CNN
-F 1 "500" V 3784 2600 50  0000 C CNN
+F 1 "1k2" V 3784 2600 50  0000 C CNN
 F 2 "Resistor_SMD:R_0805_2012Metric" V 3830 2600 50  0001 C CNN
 F 3 "~" H 3900 2600 50  0001 C CNN
@@
 L Device:LED D5
 U 1 1 60ADEA1D
-P 4300 1000
-F 0 "D5" V 4339 882 50  0000 R CNN
-F 1 "LED" V 4248 882 50  0000 R CNN
-F 2 "LED_THT:LED_D3.0mm" H 4300 1000 50  0001 C CNN
-F 3 "~" H 4300 1000 50  0001 C CNN
-	1    4300 1000
+P 4100 1000
+F 0 "D5" V 4139 882 50  0000 R CNN
+F 1 "LED Yellow" V 4048 882 50  0000 R CNN
+F 2 "LED_THT:LED_D3.0mm" H 4100 1000 50  0001 C CNN
+F 3 "~" H 4100 1000 50  0001 C CNN
+	1    4100 1000
 	0    -1   -1   0
 $EndComp
 Wire Wire Line
-	3900 1450 3900 1550
+	3700 1450 3700 1550
 $Comp
 L Device:R R19
 U 1 1 60B23E91
-P 4300 1350
-F 0 "R19" V 4093 1350 50  0000 C CNN
-F 1 "200" V 4184 1350 50  0000 C CNN
-F 2 "Resistor_SMD:R_0805_2012Metric" V 4230 1350 50  0001 C CNN
-F 3 "~" H 4300 1350 50  0001 C CNN
-	1    4300 1350
-	1    0    0    -1
-$EndComp
-Wire Wire Line
-	3900 1000 3900 1100
-Wire Wire Line
-	4300 1500 4300 1550
-Wire Wire Line
-	4300 1550 3900 1550
-Connection ~ 3900 1550
-Wire Wire Line
-	3900 1550 3900 1600
-Wire Wire Line
-	4300 1200 4300 1150
-Wire Wire Line
-	4300 850  4300 800
-Wire Wire Line
-	4300 800  4100 800
-Wire Wire Line
-	4100 800  4100 1100
-Wire Wire Line
-	4100 1100 3900 1100
-Connection ~ 3900 1100
-Wire Wire Line
-	3900 1100 3900 1150
+P 4100 1350
+F 0 "R19" V 3893 1350 50  0000 C CNN
+F 1 "2k" V 3984 1350 50  0000 C CNN
+F 2 "Resistor_SMD:R_0805_2012Metric" V 4030 1350 50  0001 C CNN
+F 3 "~" H 4100 1350 50  0001 C CNN
+	1    4100 1350
+	1    0    0    -1
+$EndComp
+Wire Wire Line
+	3700 1000 3700 1100
+Wire Wire Line
+	4100 1500 4100 1550
+Wire Wire Line
+	4100 1550 3700 1550
+Connection ~ 3700 1550
+Wire Wire Line
+	3700 1550 3700 1600
+Wire Wire Line
+	4100 1200 4100 1150
+Wire Wire Line
+	4100 850  4100 800
+Wire Wire Line
+	4100 800  3900 800
+Wire Wire Line
+	3900 800  3900 1100
+Wire Wire Line
+	3900 1100 3700 1100
+Connection ~ 3700 1100
+Wire Wire Line
+	3700 1100 3700 1150
 Wire Wire Line
 	6650 5650 6900 5650
@@
 Wire Wire Line
 	3250 3350 3200 3350
+Text GLabel 3150 3500 0    50   Input ~ 0
+GPIO13
+Wire Wire Line
+	3150 3500 3250 3500
+Wire Wire Line
+	3250 3500 3250 3350
+Connection ~ 3250 3350
 $EndSCHEMATC
